File: Hardware/DC33_Cnet_Badge_SAO/DC33_Cnet_Badge_SAO.kicad_sch (KiCad schematic)
At the start: 4 parts, among them J1 Conn_02x03_Top_Bottom

Commit message: SAO Updates
Parts:
- removed D3: LED, LED_THT:LED_D3.0mm, symbol Device:LED
- J1: footprint DC31_Cnet_Badge_SAO:PinSocket_2x03_P2.54mm_Vertical_Tab -> CactusCon_2025_CNet_SAO:PinSocket_2x03_P2.54mm_Vertical_Tab
Other:
- moved on the sheet: D1, D2
