File: Hardware/DC33_Cnet_Badge_Main/DC33_Cnet_Badge_Main.kicad_pcb (KiCad board)
At the start: 2 copper layers, 101 x 58 mm, 7 parts, among them J1 DC33_Cnet_Badge_SAO_Socket

Commit message: Added 3D models
Parts:
- added REF**: DC33_Cnet_Badge_LoRa_Antenna, DC33_Cnet_Badge_Main:DC33_Cnet_Badge_LoRa_Antenna, B.Cu at (192.5, 56.0)
Changed lines of the file:
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@@
 			(pintype "input")
+		)
+		(model "C:/Users/jgranat/My Drive/Dev/Arduino/DC33_Cnet_Badge/Hardware/3D Models/Vibra1.step"
+			(offset
+				(xyz 0 0 0)
+			)
+			(scale
+				(xyz 1 1 1)
+			)
+			(rotate
+				(xyz 0 0 180)
+			)
 		)
 	)
@@
 			(pintype "input")
 		)
+		(model "C:/Users/jgranat/My Drive/Dev/Arduino/DC33_Cnet_Badge/Hardware/3D Models/Buzz1.step"
+			(offset
+				(xyz 0 0 0)
+			)
+			(scale
+				(xyz 1 1 1)
+			)
+			(rotate
+				(xyz 0 0 90)
+			)
+		)
 	)
 	(footprint "DC33_Cnet_Badge_Main:DC33_Cnet_Badge_HiLetgo_GPS_Ant"
@@
 			)
 		)
+		(model "C:/Users/jgranat/My Drive/Dev/Arduino/DC33_Cnet_Badge/Hardware/3D Models/HiLetGo_GPS_Antenna.step"
+			(offset
+				(xyz 0 0 0)
+			)
+			(scale
+				(xyz 1 1 1)
+			)
+			(rotate
+				(xyz 0 0 0)
+			)
+		)
 	)
 	(footprint "DC33_Cnet_Badge_Main:DC33_Cnet_Badge_Heltec_V3_LoRa"
@@
 			(pintype "power_in")
 		)
+		(model "C:/Users/jgranat/My Drive/Dev/Arduino/DC33_Cnet_Badge/Hardware/Heltec V3 LoRa/heltec-wifi-lora-32-shield-1.snapshot.2/heltec_wifi_32_asm2.STEP"
+			(offset
+				(xyz 0 2.5 2.5)
+			)
+			(scale
+				(xyz 1 1 1)
+			)
+			(rotate
+				(xyz -90 0 -90)
+			)
+		)
 	)
 	(footprint "DC33_Cnet_Badge_Main:DC33_Cnet_Badge_HiLetgo_GPS"
@@
 			(pintype "power_in")
 		)
+		(model "C:/Users/jgranat/My Drive/Dev/Arduino/DC33_Cnet_Badge/Hardware/3D Models/HiLetGo_GPS_Module.step"
+			(offset
+				(xyz 0 0 1.5)
+			)
+			(scale
+				(xyz 1 1 1)
+			)
+			(rotate
+				(xyz 0 0 0)
+			)
+		)
 	)
 	(footprint "DC33_Cnet_Badge_Main:DC33_Cnet_Badge_LiPo"
@@
 			)
 		)
+		(model "C:/Users/jgranat/My Drive/Dev/Arduino/DC33_Cnet_Badge/Hardware/3D Models/LiPo.step"
+			(offset
+				(xyz 0 0 5.5)
+			)
+			(scale
+				(xyz 1 1 1)
+			)
+			(rotate
+				(xyz 0 0 90)
+			)
+		)
+	)
+	(footprint "DC33_Cnet_Badge_Main:DC33_Cnet_Badge_LoRa_Antenna"
+		(layer "B.Cu")
+		(at 192.5 56 180)
+		(property "Reference" "REF**"
+			(at 0 0.5 0)
+			(unlocked yes)
+			(layer "B.SilkS")
+			(effects
+				(font
+					(size 1 1)
+					(thickness 0.1)
+				)
+				(justify mirror)
+			)
+		)
+		(property "Value" "DC33_Cnet_Badge_LoRa_Antenna"
+			(at 0 -1 0)
+			(unlocked yes)
+			(layer "B.Fab")
+			(effects
+				(font
+					(size 1 1)
+					(thickness 0.15)
+				)
+				(justify mirror)
+			)
+		)
+		(property "Footprint" "DC33_Cnet_Badge_Main:DC33_Cnet_Badge_LoRa_Antenna"
+			(at 0 0 0)
+			(unlocked yes)
+			(layer "B.Fab")
+			(hide yes)
+			(effects
+				(font
+					(size 1 1)
+					(thickness 0.15)
+				)
+				(justify mirror)
+			)
+		)
+		(property "Datasheet" ""
+			(at 0 0 0)
+			(unlocked yes)
+			(layer "B.Fab")
+			(hide yes)
+			(effects
+				(font
+					(size 1 1)
+					(thickness 0.15)
+				)
+				(justify mirror)
+			)
+		)
+		(property "Description" ""
+			(at 0 0 0)
+			(unlocked yes)
+			(layer "B.Fab")
+			(hide yes)
+			(effects
+				(font
+					(size 1 1)
+					(thickness 0.15)
+				)
+				(justify mirror)
+			)
+		)
+		(attr smd)
+		(fp_text user "${REFERENCE}"
+			(at 0 -2.5 0)
+			(unlocked yes)
+			(layer "B.Fab")
+			(effects
+				(font
+					(size 1 1)
+					(thickness 0.15)
+				)
+				(justify mirror)
+			)
+		)
+		(model "C:/Users/jgranat/My Drive/Dev/Arduino/DC33_Cnet_Badge/Hardware/3D Models/LoRa_Antenna.step"
+			(offset
+				(xyz 28 -6 6)
+			)
+			(scale
+				(xyz 1 1 1)
+			)
+			(rotate
+				(xyz 0 0 0)
+			)
+		)

Commit message: Case_1 Files
Connections:
- J1 pad 3: unconnected-(J1-SDA-Pad3) -> Net-(J1-SDA)
- J1 pad 4: unconnected-(J1-SCL-Pad4) -> Net-(BUZZ1-POS)
- J1 pad 5: unconnected-(J1-GPIO1-Pad5) -> Net-(GPS1-RX)
- J1 pad 6: unconnected-(J1-GPIO2-Pad6) -> Net-(GPS1-TX)
- U1 pad 31: Net-(U1-GPIO45) -> Net-(J1-SDA)
- VIBRA1 pad 1: Net-(U1-GPIO45) -> Net-(J1-SDA)
Routing:
- net Net-(J1-SDA): track 0.00 -> 71.3 mm
- net Net-(U1-GPIO45): track 47.6 -> 0.00 mm
- net Net-(BUZZ1-POS): track 47.0 -> 74.2 mm
- net Net-(GPS1-RX): track 36.7 -> 60.0 mm
- net Net-(GPS1-TX): track 43.7 -> 59.6 mm
- net 3V3: track 112.9 -> 99.8 mm

Commit message: Case updates
Parts:
- moved J1 0.35 mm to (192.8, 78.0)
Routing:
- net 3V3: track 99.8 -> 99.1 mm
Changed lines of the file:
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@@
 	(footprint "DC33_Cnet_Badge_Main:DC33_Cnet_Badge_SAO_Socket"
 		(layer "F.Cu")
-		(at 192.8 77.62)
+		(at 192.8 77.975)
 		(descr "Through hole straight socket strip, 2x03, 2.54mm pitch, double cols (from Kicad 4.0.7), script generated")
 		(tags "Through hole socket strip THT 2x03 2.54mm double row")
@@
 	)
 	(segment
-		(start 186.1 68.5)
-		(end 186.1 76)
+		(start 178.5 60.9)
+		(end 178.5 57.88)
 		(width 0.2)
 		(layer "B.Cu")
@@
 	)
 	(segment
-		(start 178.5 60.9)
-		(end 186.1 68.5)
+		(start 190.26 80.515)
+		(end 186.1 76.355)
 		(width 0.2)
 		(layer "B.Cu")
@@
 	)
 	(segment
-		(start 178.5 57.88)
+		(start 186.1 68.5)
 		(end 178.5 60.9)
 		(width 0.2)
@@
 	)
 	(segment
-		(start 186.1 76)
-		(end 190.26 80.16)
+		(start 186.1 76.355)
+		(end 186.1 68.5)
 		(width 0.2)
 		(layer "B.Cu")
@@
 	(segment
 		(start 196.2 87.7)
-		(end 196.2 78.2)
+		(end 196.2 79.2)
 		(width 0.2)
 		(layer "F.Cu")
@@
 	)
 	(segment
-		(start 196.2 78.2)
-		(end 195.6 77.6)
+		(start 183.51 90.69)
+		(end 193.21 90.69)
 		(width 0.2)
 		(layer "F.Cu")
@@
 	)
 	(segment
-		(start 195.6 77.6)
-		(end 195.58 77.62)
+		(start 151.2 65.6)
+		(end 151.2 68.2)
+		(width 0.2)
+		(layer "F.Cu")
+		(net 3)
+	)
+	(segment
+		(start 182.29 90.69)
+		(end 183.51 90.69)
+		(width 0.2)
+		(layer "F.Cu")
+		(net 3)
+	)
+	(segment
+		(start 151.2 68.2)
+		(end 160.5 77.5)
+		(width 0.2)
+		(layer "F.Cu")
+		(net 3)
+	)
+	(segment
+		(start 126.4 56.64)
+		(end 129.26 59.5)
+		(width 0.2)
+		(layer "F.Cu")
+		(net 3)
+	)
+	(segment
+		(start 169.1 77.5)
+		(end 182.29 90.69)
+		(width 0.2)
+		(layer "F.Cu")
+		(net 3)
+	)
+	(segment
+		(start 196.2 79.2)
+		(end 194.975 77.975)
+		(width 0.2)
+		(layer "F.Cu")
+		(net 3)
+	)
+	(segment
+		(start 160.5 77.5)
+		(end 169.1 77.5)
+		(width 0.2)
+		(layer "F.Cu")
+		(net 3)
+	)
+	(segment
+		(start 194.975 77.975)
+		(end 192.8 77.975)
+		(width 0.2)
+		(layer "F.Cu")
+		(net 3)
+	)
+	(segment
+		(start 129.26 59.5)
+		(end 145.1 59.5)
 		(width 0.2)
 		(layer "F.Cu")
@@
 	)
 	(segment
-		(start 151.2 65.6)
-		(end 151.2 68.2)
-		(width 0.2)
-		(layer "F.Cu")
-		(net 3)
-	)
-	(segment
-		(start 182.29 90.69)
-		(end 183.51 90.69)
-		(width 0.2)
-		(layer "F.Cu")
-		(net 3)
-	)
-	(segment
-		(start 151.2 68.2)
-		(end 160.5 77.5)
-		(width 0.2)
-		(layer "F.Cu")
-		(net 3)
-	)
-	(segment
-		(start 126.4 56.64)
-		(end 129.26 59.5)
-		(width 0.2)
-		(layer "F.Cu")
-		(net 3)
-	)
-	(segment
-		(start 169.1 77.5)
-		(end 182.29 90.69)
-		(width 0.2)
-		(layer "F.Cu")
-		(net 3)
-	)
-	(segment
-		(start 183.51 90.69)
-		(end 193.21 90.69)
-		(width 0.2)
-		(layer "F.Cu")
-		(net 3)
-	)
-	(segment
-		(start 160.5 77.5)
-		(end 169.1 77.5)
-		(width 0.2)
-		(layer "F.Cu")
-		(net 3)
-	)
-	(segment
-		(start 129.26 59.5)
-		(end 145.1 59.5)
-		(width 0.2)
-		(layer "F.Cu")
-		(net 3)
-	)
-	(segment
-		(start 195.58 77.62)
-		(end 192.8 77.62)
-		(width 0.2)
-		(layer "F.Cu")
-		(net 3)
-	)
-	(segment
 		(start 145.1 59.5)
 		(end 151.2 65.6)
@@
 	)
 	(segment
-		(start 192.8 82.7)
-		(end 192.8 88.106346)
+		(start 192.8 88.106346)
+		(end 183.986346 96.92)
 		(width 0.2)
 		(layer "B.Cu")
@@
 	)
 	(segment
-		(start 192.8 88.106346)
-		(end 183.986346 96.92)
+		(start 183.986346 96.92)
+		(end 183.02 96.92)
 		(width 0.2)
 		(layer "B.Cu")
@@
 	)
 	(segment
-		(start 183.986346 96.92)
-		(end 183.02 96.92)
+		(start 192.8 88.106346)
+		(end 192.8 83.055)
 		(width 0.2)
 		(layer "B.Cu")
@@
 	)
 	(segment
-		(start 190.26 82.7)
-		(end 190.26 89.02)
+		(start 190.26 89.02)
+		(end 190.26 83.055)
 		(width 0.2)
 		(layer "B.Cu")
@@
 	)
 	(segment
-		(start 188.496346 74.23)
-		(end 191.65 77.383654)
+		(start 192.8 80.515)
+		(end 192.8 80.3)
 		(width 0.2)
 		(layer "F.Cu")
@@
 	)
 	(segment
-		(start 191.65 77.383654)
-		(end 191.65 79.01)
+		(start 192.8 80.3)
+		(end 191.41 78.91)
 		(width 0.2)
 		(layer "F.Cu")
@@
 	)
 	(segment
-		(start 191.65 79.01)
-		(end 192.8 80.16)
+		(start 191.41 77.143654)
+		(end 188.496346 74.23)
 		(width 0.2)
 		(layer "F.Cu")
@@
 		(width 0.2)
 		(layer "F.Cu")
+		(net 6)
+	)
+	(segment
+		(start 191.41 78.91)
+		(end 191.41 77.143654)
+		(width 0.2)
+		(layer "F.Cu")

Commit message: Updated case
Parts:
- moved J1 28.3 mm to (210.0, 100.4)
Routing:
- net Net-(BUZZ1-POS): track 74.5 -> 109.0 mm
- net Net-(J1-SDA): track 71.7 -> 97.9 mm, vias 0 -> 2
- net Net-(GPS1-RX): track 59.6 -> 81.9 mm
- net 3V3: track 99.1 -> 111.4 mm
- net Net-(GPS1-TX): track 59.2 -> 68.9 mm
Other:
- outline, holes or cut-outs redrawn

Commit message: Updated PCB
Parts:
- added REF**: DC33_Logo, DC33_Cnet_Badge_Main:DC33_Logo, B.Cu at (183.5, 74.5)
- added REF**: CompuNet PCB Logo, DC33_Cnet_Badge_Main:CompuNet PCB Logo, B.Cu at (159.5, 66.0)
- added SW1: PB_Switch, DC33_Cnet_Badge_Main:PB_Switch, B.Cu at (201.2, 103.0)
Connections:
- J1 pad 4: Net-(BUZZ1-POS) -> Net-(J1-SCL)
- J1 pad 5: Net-(GPS1-RX) -> Net-(J1-GPIO1)
- J1 pad 6: Net-(GPS1-TX) -> Net-(J1-GPIO2)
- U1 pad 27: unconnected-(U1-GPIO39-Pad27) -> Net-(J1-GPIO2)
- U1 pad 28: unconnected-(U1-GPIO40-Pad28) -> Net-(J1-GPIO1)
- U1 pad 29: unconnected-(U1-GPIO41-Pad29) -> Net-(J1-SCL)
- U1 pad 30: unconnected-(U1-GPIO42-Pad30) -> Net-(J1-SDA)
- U1 pad 31: Net-(J1-SDA) -> Net-(U1-GPIO45)
- VIBRA1 pad 1: Net-(J1-SDA) -> Net-(U1-GPIO45)
Routing:
- net Net-(J1-SCL): track 0.00 -> 188.0 mm
- net Net-(J1-GPIO1): track 0.00 -> 186.0 mm, vias 0 -> 2
- net Net-(J1-GPIO2): track 0.00 -> 172.2 mm, vias 0 -> 1
- net Net-(J1-SDA): track 97.9 -> 178.1 mm, vias 2 -> 0
- net Net-(BUZZ1-POS): track 109.0 -> 46.5 mm
- net Net-(GPS1-RX): track 81.9 -> 36.4 mm
- net Net-(U1-GPIO45): track 0.00 -> 43.2 mm
- net Net-(GPS1-TX): track 68.9 -> 33.4 mm
- net 3V3: track 111.4 -> 122.6 mm
Other:
- board text added: "@slash128"
- board text added: "https://github.com/slash128v6/DC33_Cnet_Badge"

Commit message: Updated PCB
Parts:
- moved J1 4.89 mm to (214.9, 100.4)
- moved SW1 4.75 mm to (206.0, 103.0)
Routing:
- net Net-(J1-GPIO2): track 172.2 -> 177.2 mm
- net 3V3: track 122.6 -> 127.0 mm
- net Net-(J1-GPIO1): track 186.0 -> 190.3 mm
- net Net-(J1-SCL): track 188.0 -> 192.2 mm
- net Net-(J1-SDA): track 178.1 -> 180.2 mm
Other:
- board size 101 x 58 mm -> 105.5 x 58 mm

Commit message: Latest updates
Parts:
- SW1: value PB_Switch -> Tactile_Switch; footprint DC33_Cnet_Badge_Main:PB_Switch -> DC33_Cnet_Badge_Main:Tactile_Switch-13mm; moved to F.Cu
- moved SW1 39.6 mm to (178.5, 74.5), turned to 180 degrees
- moved J1 28.0 mm to (193.4, 82.5)
- moved VIBRA1 13.3 mm to (190.1, 68.2), turned to -90 degrees
- moved REF** 5.03 mm to (178.5, 74.5)
- moved GPS_ANT 3.50 mm to (137.5, 94.5)
- moved GPS1 2.00 mm to (169.0, 94.5)
- moved REF** 1.95 mm to (157.6, 66.0)
Routing:
- net Net-(J1-SCL): track 192.2 -> 65.4 mm
- net Net-(J1-GPIO1): track 190.3 -> 65.3 mm, vias 2 -> 0
- net Net-(J1-GPIO2): track 177.2 -> 63.3 mm, vias 1 -> 0
- net Net-(J1-SDA): track 180.2 -> 71.2 mm
- net Net-(U1-GPIO45): track 43.2 -> 67.8 mm
- net 3V3: track 127.0 -> 109.7 mm
- net GND: track 0.00 -> 16.4 mm
- net Net-(GPS1-TX): track 33.4 -> 35.4 mm
- net Net-(GPS1-RX): track 36.4 -> 38.4 mm
Other:
- board size 105.5 x 58 mm -> 101 x 58 mm
