File: Hardware/DC33_Cnet_Badge_Main/DC33_Cnet_Badge_Main.kicad_sch (KiCad schematic)
At the start: 5 parts, among them J1 DC33_Cnet_Badge_SAO_Socket

Commit message: Case_1 Files
Connections:
- net at GPS1.2 (RX), U1.13 (GPIO47): now also J1.5 (GPIO1)
- net at GPS1.3 (TX), U1.14 (GPIO48): now also J1.6 (GPIO2)
- net at J1.3 (SDA): now also U1.31 (GPIO45), VIBRA1.1 (POS)
- net at J1.4 (SCL): now also BUZZ1.1 (POS), U1.32 (GPIO46)
Changed lines of the file:
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@@
 	(generator_version "8.0")
 	(paper "A4")
+	(junction
+		(at 109.22 104.14)
+		(diameter 0)
+		(color 0 0 0 0)
+	)
+	(junction
+		(at 177.8 87.63)
+		(diameter 0)
+		(color 0 0 0 0)
+	)
+	(junction
+		(at 173.99 83.82)
+		(diameter 0)
+		(color 0 0 0 0)
+	)
+	(junction
+		(at 101.6 106.68)
+		(diameter 0)
+		(color 0 0 0 0)
+	)
+	(wire
+		(pts
+			(xy 177.8 87.63) (xy 157.48 87.63)
+		)
+		(stroke
+			(width 0)
+			(type default)
+		)
+	)
 	(wire
 		(pts
@@
 	(wire
 		(pts
+			(xy 170.18 44.45) (xy 182.88 44.45)
+		)
+		(stroke
+			(width 0)
+			(type default)
+		)
+	)
+	(wire
+		(pts
+			(xy 182.88 44.45) (xy 182.88 24.13)
+		)
+		(stroke
+			(width 0)
+			(type default)
+		)
+	)
+	(wire
+		(pts
 			(xy 157.48 44.45) (xy 151.13 44.45)
 		)
@@
 	(wire
 		(pts
-			(xy 144.78 83.82) (xy 190.5 83.82)
+			(xy 144.78 83.82) (xy 173.99 83.82)
 		)
 		(stroke
@@
 	(wire
 		(pts
-			(xy 190.5 87.63) (xy 157.48 87.63)
+			(xy 173.99 83.82) (xy 190.5 83.82)
+		)
+		(stroke
+			(width 0)
+			(type default)
+		)
+	)
+	(wire
+		(pts
+			(xy 190.5 87.63) (xy 177.8 87.63)
+		)
+		(stroke
+			(width 0)
+			(type default)
+		)
+	)
+	(wire
+		(pts
+			(xy 101.6 24.13) (xy 101.6 106.68)
 		)
 		(stroke
@@
 	(wire
 		(pts
+			(xy 101.6 106.68) (xy 95.25 106.68)
+		)
+		(stroke
+			(width 0)
+			(type default)
+		)
+	)
+	(wire
+		(pts
 			(xy 157.48 87.63) (xy 157.48 86.36)
 		)
@@
 	(wire
 		(pts
+			(xy 170.18 46.99) (xy 177.8 46.99)
+		)
+		(stroke
+			(width 0)
+			(type default)
+		)
+	)
+	(wire
+		(pts
+			(xy 157.48 49.53) (xy 109.22 49.53)
+		)
+		(stroke
+			(width 0)
+			(type default)
+		)
+	)
+	(wire
+		(pts
 			(xy 190.5 80.01) (xy 186.69 80.01)
 		)
@@
 	(wire
 		(pts
+			(xy 182.88 24.13) (xy 101.6 24.13)
+		)
+		(stroke
+			(width 0)
+			(type default)
+		)
+	)
+	(wire
+		(pts
 			(xy 77.47 88.9) (xy 60.96 88.9)
 		)
@@
 	(wire
 		(pts
+			(xy 177.8 46.99) (xy 177.8 87.63)
+		)
+		(stroke
+			(width 0)
+			(type default)
+		)
+	)
+	(wire
+		(pts
 			(xy 105.41 114.3) (xy 105.41 99.06)
 		)
@@
 	(wire
 		(pts
-			(xy 114.3 104.14) (xy 63.5 104.14)
+			(xy 170.18 49.53) (xy 173.99 49.53)
+		)
+		(stroke
+			(width 0)
+			(type default)
+		)
+	)
+	(wire
+		(pts
+			(xy 109.22 49.53) (xy 109.22 104.14)
+		)
+		(stroke
+			(width 0)
+			(type default)
+		)
+	)
+	(wire
+		(pts
+			(xy 109.22 104.14) (xy 63.5 104.14)
+		)
+		(stroke
+			(width 0)
+			(type default)
+		)
+	)
+	(wire
+		(pts
+			(xy 114.3 104.14) (xy 109.22 104.14)
 		)
 		(stroke
@@
 	(wire
 		(pts
+			(xy 173.99 49.53) (xy 173.99 83.82)
+		)
+		(stroke
+			(width 0)
+			(type default)
+		)
+	)
+	(wire
+		(pts
 			(xy 190.5 91.44) (xy 181.61 91.44)
 		)
@@
 	(wire
 		(pts
-			(xy 114.3 106.68) (xy 95.25 106.68)
-		)
-		(stroke
+			(xy 114.3 106.68) (xy 101.6 106.68)
+		)
+		(stroke

Commit message: Updated PCB
Parts:
- added SW1: PB_Switch, DC33_Cnet_Badge_Main:PB_Switch, symbol DC33_Cnet_Badge:PB_Switch
Connections:
- net GND: now also SW1.2
- net at GPS1.2 (RX), U1.13 (GPIO47): no longer J1.5 (GPIO1)
- net at GPS1.3 (TX), U1.14 (GPIO48): no longer J1.6 (GPIO2)
- net at U1.31 (GPIO45), VIBRA1.1 (POS): no longer J1.3 (SDA)
- net at BUZZ1.1 (POS), U1.32 (GPIO46): no longer J1.4 (SCL)
- net at U1.27 (GPIO39): now also J1.6 (GPIO2)
- net at U1.28 (GPIO40): now also J1.5 (GPIO1), SW1.1
- net at U1.29 (GPIO41): now also J1.4 (SCL)
- net at U1.30 (GPIO42): now also J1.3 (SDA)

Commit message: Latest updates
Parts:
- removed SW1: PB_Switch, DC33_Cnet_Badge_Main:PB_Switch, symbol DC33_Cnet_Badge:PB_Switch
- added SW1: Tactile_Switch, DC33_Cnet_Badge_Main:Tactile_Switch-13mm, symbol DC33_Cnet_Badge:Tactile_Switch
Connections:
- net GND: now also SW1.2
- net at J1.5 (GPIO1), U1.28 (GPIO40): now also SW1.1
